File: LED_Board.kicad_pcb (KiCad board)
At the start: 2 copper layers, 74.2 x 75.1 mm, 25 parts, among them Q4 AO3400A

Commit message: Release 2
Connections:
- D1 pad 3: GND -> unconnected-(D1-PAD-Pad3)
Routing:
- net GND: track 3.10 -> 0.00 mm, vias 3 -> 0
